File: schematic/led_clock.kicad_pcb (KiCad board)
At the start: 2 copper layers, 24 parts, among them J3 CONN_01X04, J4 CONN_01X04, J5 USB_OTG, J6 CONN_01X03, U1 SN74LVC2T45, U2 Nucleo32, U3 PCF8563, U4 MCP9701

Commit message: Rev 1.0 of circuit boards
Parts:
- removed C4, C5: 6p, Capacitors_SMD:C_0603
- removed C6: 0.1u, Capacitors_SMD:C_0603
- removed D1: D, Diodes_SMD:D_0603
- removed R4, R5: 4.7k, Resistors_SMD:R_0603
- removed U3: PCF8563, Housings_SOIC:SOIC-8-1EP_3.9x4.9mm_Pitch1.27mm
- added C10: 0.1u, Capacitors_SMD:C_0603, F.Cu at (171.4, 111.1)
- added C11: 0.1u, Capacitors_SMD:C_0603, F.Cu at (168.9, 111.1)
- added J7: CONN_01X02, Pin_Headers:Pin_Header_Straight_1x02_Pitch2.54mm, F.Cu at (178.1, 101.2)
- added U5: SN74LVC1T45, TO_SOT_Packages_SMD:SOT-23-6, F.Cu at (170.2, 114.9)
- J6: footprint Pin_Headers:Pin_Header_Angled_1x03_Pitch2.54mm -> Pin_Headers:Pin_Header_Straight_1x03_Pitch2.54mm
- U1: value SN74LVC2T45 -> SN74LVC1T45; footprint Housings_SSOP:MSOP-8_3x3mm_Pitch0.65mm -> TO_SOT_Packages_SMD:SOT-23-6
- moved J5 61.4 mm to (185.7, 102.4), turned to 90 degrees
- moved R6 51.9 mm to (178.8, 97.3), turned to 180 degrees
- moved C3 29.2 mm to (170.2, 101.6)
- moved J6 24.0 mm to (152.7, 134.9), turned to 270 degrees
- moved U4 23.3 mm to (164.3, 134.4)
- moved R1 21.4 mm to (149.9, 120.4), turned to 270 degrees
- moved C8 14.7 mm to (157.2, 134.4), turned to 270 degrees
- moved R2 10.5 mm to (172.7, 130.8), turned to 180 degrees
- moved C2 9.01 mm to (159.3, 117.3)
- moved J3 7.62 mm to (184.2, 120.7), turned to 0 degrees
- moved U2 7.24 mm to (154.3, 103.5)
- moved C1 7.24 mm to (159.4, 98.4)
- moved C7 4.62 mm to (168.9, 123.8), turned to 90 degrees
- moved R3 4.58 mm to (172.7, 118.1), turned to 180 degrees
- moved C9 4.49 mm to (171.4, 123.8), turned to 90 degrees
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Connections:
- J3 pad 1: Net-(J3-Pad1) -> GND
- J3 pad 2: DS_DAT -> +5V
- J3 pad 3: +5V -> DS_DAT
- J3 pad 4: GND -> Net-(J3-Pad4)
- U1 pad 2: PIX_DAT -> GND
- U1 pad 3: PIX_CLK -> PIX_DAT
- U1 pad 4: GND -> DS_DAT
- U1 pad 6: DS_CLK -> +5V
Routing:
- net PIX_DIR: track 0.00 -> 60.0 mm, vias 0 -> 3
- net GND: track 0.00 -> 43.2 mm, vias 0 -> 15
- net LUX: track 0.00 -> 26.1 mm
- net PIX_DAT: track 0.00 -> 25.4 mm
- net TEMP: track 0.00 -> 23.2 mm, vias 0 -> 1
- net Net-(J5-Pad6): track 0.00 -> 19.2 mm
- net PIX_CLK: track 0.00 -> 16.9 mm, vias 0 -> 1
- net +5V: track 3.02 -> 15.9 mm, vias 0 -> 1
- net +3V3: track 3.29 -> 14.4 mm, vias 0 -> 1
- net DS_CLK: track 10.4 -> 15.6 mm
- net DS_DAT: track 15.1 -> 16.4 mm, vias 1 -> 0
- added copper zone on F.Cu, net +3V3
- added copper zone on F.Cu, net +5V
- added copper zone on B.Cu, net GND
Other:
- board outline added: 44.4 x 46.7 mm
- board text added: "DotStar LED Clock Rev 1.0"
